Commit message: modified

File: robots/descriptions/go2_description/xacro/gps.xacro (robot description, xacro)
@@ -23,5 +23,5 @@
   <!-- trunkに固定 -->
   <joint name="gps_joint" type="fixed">
-    <parent link="trunk"/>
+    <parent link="base_link"/>
     <child link="gps_link"/>
     <!-- 上にちょっと乗せる -->

File: robots/descriptions/go2_description/xacro/robot.xacro (robot description, xacro)
@@ -57,5 +57,5 @@
     </link>
     <joint name="imu_joint" type="fixed">
-        <parent link="trunk"/>
+        <parent link="base_link"/>
         <child link="imu_link"/>
         <origin rpy="0 0 0" xyz="0 0 0"/>

File: robots/descriptions/go2_description/xacro/robot_VLP.xacro (robot description, xacro)
@@ -57,5 +57,5 @@
     </link>
     <joint name="imu_joint" type="fixed">
-        <parent link="trunk"/>
+        <parent link="base_link"/>
         <child link="imu_link"/>
         <origin rpy="0 0 0" xyz="0 0 0"/>
